File: SchematicHandroute.brd (EAGLE design)
At the start: 84 x 96 mm, 64 parts

Commit message: 013120meeting
Parts:
- moved LED_LOW_BAT 33.5 mm to (33.0, 44.5)
- moved R14 30.7 mm to (30.5, 47.0)
- moved R5 15.2 mm to (47.0, 78.7), turned to 0 degrees
- moved R4 2.84 mm to (3.81, 57.1)
- moved C10 2.54 mm to (40.6, 48.3)
- moved C6 2.54 mm to (36.8, 48.3)
- moved R8 1.80 mm to (8.89, 58.2)
Routing:
- net +3V3: track 0.00 -> 166.4 mm
- net N$1: track 0.00 -> 70.0 mm
- net B1: track 0.00 -> 54.4 mm
- net N$4: track 0.00 -> 47.1 mm
- net B0: track 0.00 -> 44.3 mm
- net LMTR+: track 0.00 -> 34.0 mm
- net +5V: track 0.00 -> 33.2 mm
- net LMTR-: track 0.00 -> 25.6 mm
- net N$14: track 0.00 -> 23.9 mm, vias 0 -> 2
- net GND: track 0.00 -> 22.4 mm
- net NRST: track 0.00 -> 17.1 mm
- net N$3: track 0.00 -> 16.7 mm
- net N$2: track 0.00 -> 16.1 mm
- net V+: track 0.00 -> 14.5 mm
- net N$9: track 0.00 -> 9.04 mm
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- added copper zone on layer 1, net GND
- added copper zone on layer 16, net GND
