File: SchematicHandroute.sch (EAGLE design)
At the start: 35 parts

Commit message: 013120meeting
Parts:
- added B0, B1: POLOLU_BUTTON, POLOLU_BUTTON:POLOLU_BUTTON
- added C12, C13: 1.0uF, CAP_CERAMIC_0805IN_2012MM:CAP_CERAMIC_0805IN_2012MM
- added LED-PWR, LED1, LED2, LED3, LED_LOW_BAT: LED, LED_0805:LED
- added MTR_L, MTR_R: MOTOR_ENCODER_HEADER, MOTOR_ENCODER_HEADER:MOTOR_ENCODER_HEADER
- added R10: 10K, RESISTOR_0805IN_2012MM:RESISTOR_0805IN_2012MM
- added R11, R12, R13, R14, R15: 1K, RESISTOR_0805IN_2012MM:RESISTOR_0805IN_2012MM
- added R16, R17, R18, R19, R20, R21: 47K, RESISTOR_0805IN_2012MM:RESISTOR_0805IN_2012MM
- added R22: 30K, RESISTOR_0805IN_2012MM:RESISTOR_0805IN_2012MM
- added TC4427_L, TC4427_R: TC4427_SOIC8, TC4427:TC4427_SOIC8
- added ZXMHC3_L, ZXMHC3_R: ZXMHC3, ZXMHC3:ZXMHC3
Connections:
- removed net BO: STM32F1.PB0
- removed net LPWN_B: STM32F1.PB8
- removed net N$10: R5.2, RE_LF.E
- removed net N$11: R6.2, RE_LD.E
- removed net N$12: R7.2, RE_RD.E
- removed net N$13: R8.2, RE_RF.E
- new net B0: B0.1, R16.2, STM32F1.PB0
- new net LMTR+: MTR_L.MTR_+, ZXMHC3_L.N1D/P1D
- new net LMTR-: MTR_L.MTR_-, ZXMHC3_L.N2D/P2D
- new net LPWM_B: R19.2, STM32F1.PB8, TC4427_L.IN_B
- new net N$17: TC4427_L.OUT_B, ZXMHC3_L.N2G, ZXMHC3_L.P2G
- new net N$18: TC4427_L.OUT_A, ZXMHC3_L.N1G, ZXMHC3_L.P1G
- new net N$19: TC4427_R.OUT_A, ZXMHC3_R.N1G, ZXMHC3_R.P1G
- new net N$20: TC4427_R.OUT_B, ZXMHC3_R.N2G, ZXMHC3_R.P2G
- new net N$21: LED1.C, R11.2
- new net N$22: LED2.C, R12.2
- new net N$23: LED3.C, R13.2
- new net N$24: LED_LOW_BAT.C, R14.2
- new net N$25: LED-PWR.C, R15.2
- new net RMTR+: MTR_R.MTR_+, ZXMHC3_R.N1D/P1D
- new net RMTR-: MTR_R.MTR_-, ZXMHC3_R.N2D/P2D
- net +3V3: now also B0.2, B1.2, LED-PWR.A, MTR_L.ENC_VDD, MTR_R.ENC_VDD
- net +5V: now also ZXMHC3_L.P1S/P2S, ZXMHC3_R.P1S/P2S
- net B1: now also B1.1, R17.2
- net GND: now also C12.2, C13.2, MTR_L.ENC_GND, MTR_R.ENC_GND, R10.1, R11.1, R12.1, R13.1, R14.1, R15.1, R16.1, R17.1, R18.1, R19.1, R20.1, R21.1, TC4427_L.GND, TC4427_R.GND, ZXMHC3_L.N1S/N2S, ZXMHC3_R.N1S/N2S
- net LED1: now also LED1.A
- net LED2: now also LED2.A
- net LED3: now also LED3.A
- net LED_LOW_BAT: now also LED_LOW_BAT.A
- net LENC_A: now also MTR_L.ENC_A
- net LENC_B: now also MTR_L.ENC_B
- net LPWM_A: now also R18.2, TC4427_L.IN_A
- net RENC_A: now also MTR_R.ENC_A
- net RENC_B: now also MTR_R.ENC_B
- net RE_LD: now also R6.2, RE_LD.E
- net RE_LF: now also R5.2, RE_LF.E
- net RE_RD: now also R7.2, RE_RD.E
- net RE_RF: now also R8.2, RE_RF.E
- net RPWM_A: now also R20.2, TC4427_R.IN_A
- net RPWM_B: now also R21.2, TC4427_R.IN_B
- net V+: now also C12.1, C13.1, R22.2, TC4427_L.VDD, TC4427_R.VDD
- net VOLTMETER: now also R10.2, R22.1
Other:
- note added: "Buttons"
- note added: "LEDs"
- note added: "Motor Control"
- note added: "Voltmeter"
- moved on the sheet: C1, C10, C11, C2, C3, C4, C5, C6, C7, C8, C9, COMM1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
