File: Schematic.sch (EAGLE design)
At the start: 63 parts

Commit message: error fix
Parts:
- R10: value (none) -> 10K
- R22: value (none) -> 30K
Connections:
- removed net BO: STM32F1.PB0
- removed net LPWN_B: STM32F1.PB8
- removed net N$10: R5.2, RE_LF.E
- removed net N$11: R6.2, RE_LD.E
- removed net N$12: R7.2, RE_RD.E
- removed net N$13: R8.2, RE_RF.E
- removed net VBAT: R22.2
- net B0: now also STM32F1.PB0
- net LPWM_B: now also STM32F1.PB8
- net RE_LD: now also R6.2, RE_LD.E
- net RE_LF: now also R5.2, RE_LF.E
- net RE_RD: now also R7.2, RE_RD.E
- net RE_RF: now also R8.2, RE_RF.E
- net V+: now also R22.2
Changed lines of the file:
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@@
 <part name="GND29" library="SUPPLY" deviceset="GND" device=""/>
 <part name="+3V7" library="SUPPLY" deviceset="+3V3" device=""/>
-<part name="R10" library="RESISTOR_0805IN_2012MM" deviceset="RESISTOR_0805IN_2012MM" device=""/>
-<part name="R22" library="RESISTOR_0805IN_2012MM" deviceset="RESISTOR_0805IN_2012MM" device=""/>
+<part name="R10" library="RESISTOR_0805IN_2012MM" deviceset="RESISTOR_0805IN_2012MM" device="" value="10K"/>
+<part name="R22" library="RESISTOR_0805IN_2012MM" deviceset="RESISTOR_0805IN_2012MM" device="" value="30K"/>
 <part name="GND30" library="SUPPLY" deviceset="GND" device=""/>
+<part name="VBAT4" library="SUPPLY" deviceset="VBAT" device=""/>
 </parts>
 <sheets>
@@
 <instance part="GND30" gate="1" x="246.38" y="-30.48" smashed="yes" rot="R270">
 <attribute name="VALUE" x="246.38" y="-29.21" size="1.778" layer="96"/>
+</instance>
+<instance part="VBAT4" gate="G$1" x="299.72" y="-30.48" smashed="yes" rot="R270">
+<attribute name="VALUE" x="297.18" y="-27.94" size="1.778" layer="96"/>
 </instance>
 </instances>
@@
 <junction x="99.06" y="-327.66"/>
 </segment>
+<segment>
+<pinref part="R22" gate="G$1" pin="2"/>
+<wire x1="287.02" y1="-30.48" x2="297.18" y2="-30.48" width="0.1524" layer="91"/>
+<label x="292.1" y="-30.48" size="1.778" layer="95"/>
+<pinref part="VBAT4" gate="G$1" pin="V+"/>
+</segment>
 </net>
 <net name="N$9" class="0">
@@
 <pinref part="C11" gate="G$1" pin="1"/>
 <wire x1="309.88" y1="-248.92" x2="309.88" y2="-254" width="0.1524" layer="91"/>
-<wire x1="309.88" y1="-248.92" x2="309.88" y2="-241.3" width="0.1524" layer="91"/>
+<label x="309.88" y="-243.84" size="1.778" layer="95" rot="R90"/>
+<wire x1="309.88" y1="-248.92" x2="309.88" y2="-243.84" width="0.1524" layer="91"/>
 <junction x="309.88" y="-248.92"/>
-<label x="309.88" y="-243.84" size="1.778" layer="95" rot="R90"/>
 </segment>
 <segment>
@@
 <junction x="426.72" y="-274.32"/>
 <label x="426.72" y="-271.78" size="1.778" layer="95" rot="R90"/>
-</segment>
-<segment>
-<pinref part="MTR_L" gate="G$1" pin="ENC_VDD"/>
-<pinref part="+3V4" gate="G$1" pin="+3V3"/>
-<wire x1="220.98" y1="-248.92" x2="220.98" y2="-236.22" width="0.1524" layer="91"/>
-</segment>
-<segment>
-<pinref part="MTR_R" gate="G$1" pin="ENC_VDD"/>
-<pinref part="+3V5" gate="G$1" pin="+3V3"/>
-<wire x1="220.98" y1="-320.04" x2="220.98" y2="-307.34" width="0.1524" layer="91"/>
 </segment>
 <segment>
@@
 <wire x1="220.98" y1="-109.22" x2="220.98" y2="-119.38" width="0.1524" layer="91"/>
 </segment>
+<segment>
+<pinref part="+3V4" gate="G$1" pin="+3V3"/>
+<pinref part="MTR_L" gate="G$1" pin="ENC_VDD"/>
+<wire x1="220.98" y1="-236.22" x2="220.98" y2="-248.92" width="0.1524" layer="91"/>
+</segment>
+<segment>
+<pinref part="+3V5" gate="G$1" pin="+3V3"/>
+<pinref part="MTR_R" gate="G$1" pin="ENC_VDD"/>
+<wire x1="220.98" y1="-307.34" x2="220.98" y2="-320.04" width="0.1524" layer="91"/>
+</segment>
 </net>
 <net name="TX" class="0">
@@
 <wire x1="281.94" y1="-289.56" x2="327.66" y2="-289.56" width="0.1524" layer="91"/>
 <junction x="281.94" y="-289.56"/>
-</segment>
-</net>
-<net name="N$10" class="0">
-<segment>
-<pinref part="RE_LF" gate="G$1" pin="E"/>
-<wire x1="25.4" y1="-39.37" x2="25.4" y2="-49.53" width="0.1524" layer="91"/>
-<pinref part="R5" gate="G$1" pin="2"/>
-</segment>
-</net>
-<net name="N$11" class="0">
-<segment>
-<pinref part="RE_LD" gate="G$1" pin="E"/>
-<wire x1="48.26" y1="-39.37" x2="48.26" y2="-49.53" width="0.1524" layer="91"/>
-<pinref part="R6" gate="G$1" pin="2"/>
-</segment>
-</net>
-<net name="N$12" class="0">
-<segment>
-<pinref part="RE_RD" gate="G$1" pin="E"/>
-<wire x1="67.31" y1="-38.1" x2="67.31" y2="-48.26" width="0.1524" layer="91"/>
-<pinref part="R7" gate="G$1" pin="2"/>
-</segment>
-</net>
-<net name="N$13" class="0">
-<segment>
-<pinref part="RE_RF" gate="G$1" pin="E"/>
-<wire x1="86.36" y1="-38.1" x2="86.36" y2="-48.26" width="0.1524" layer="91"/>
-<pinref part="R8" gate="G$1" pin="2"/>
 </segment>
 </net>
@@
 </segment>
 </net>
-<net name="BO" class="0">
-<segment>
-<pinref part="STM32F1" gate="G$1" pin="PB0"/>
-<wire x1="368.3" y1="-330.2" x2="368.3" y2="-340.36" width="0.1524" layer="91"/>
-<label x="368.3" y="-340.36" size="1.778" layer="95" rot="R90"/>
-</segment>
-</net>
 <net name="RENC_A" class="0">
 <segment>
@@
 </segment>
 </net>
-<net name="LPWN_B" class="0">
-<segment>
-<pinref part="STM32F1" gate="G$1" pin="PB8"/>
-<wire x1="353.06" y1="-256.54" x2="353.06" y2="-246.38" width="0.1524" layer="91"/>
-<label x="353.06" y="-248.92" size="1.778" layer="95" rot="R90"/>
-</segment>
-</net>
 <net name="RPWM_A" class="0">
 <segment>
@@
 <label x="314.96" y="-299.72" size="1.778" layer="95"/>
 </segment>
+<segment>
+<pinref part="RE_LF" gate="G$1" pin="E"/>
+<wire x1="25.4" y1="-39.37" x2="25.4" y2="-49.53" width="0.1524" layer="91"/>
+<pinref part="R5" gate="G$1" pin="2"/>
+<label x="25.4" y="-45.72" size="1.778" layer="95"/>
+</segment>
 </net>
 <net name="RE_LD" class="0">
@@
 <label x="314.96" y="-297.18" size="1.778" layer="95"/>
 </segment>
+<segment>
+<pinref part="RE_LD" gate="G$1" pin="E"/>
+<wire x1="48.26" y1="-39.37" x2="48.26" y2="-49.53" width="0.1524" layer="91"/>
+<pinref part="R6" gate="G$1" pin="2"/>
+<label x="48.26" y="-45.72" size="1.778" layer="95"/>
+</segment>
 </net>
 <net name="RE_RD" class="0">
@@
 <label x="314.96" y="-294.64" size="1.778" layer="95"/>
 </segment>
+<segment>
+<pinref part="RE_RD" gate="G$1" pin="E"/>
+<wire x1="67.31" y1="-38.1" x2="67.31" y2="-48.26" width="0.1524" layer="91"/>
+<pinref part="R7" gate="G$1" pin="2"/>
+<label x="68.58" y="-45.72" size="1.778" layer="95"/>
+</segment>
 </net>
 <net name="RE_RF" class="0">
@@
 <wire x1="327.66" y1="-292.1" x2="317.5" y2="-292.1" width="0.1524" layer="91"/>
 <label x="314.96" y="-292.1" size="1.778" layer="95"/>
+</segment>
+<segment>
+<pinref part="RE_RF" gate="G$1" pin="E"/>
+<wire x1="86.36" y1="-38.1" x2="86.36" y2="-48.26" width="0.1524" layer="91"/>
+<pinref part="R8" gate="G$1" pin="2"/>
+<label x="86.36" y="-45.72" size="1.778" layer="95"/>
 </segment>
 </net>
@@
 <junction x="38.1" y="-264.16"/>
 <label x="7.62" y="-264.16" size="1.778" layer="95"/>
+</segment>
+<segment>
+<pinref part="STM32F1" gate="G$1" pin="PB8"/>
+<wire x1="353.06" y1="-256.54" x2="353.06" y2="-246.38" width="0.1524" layer="91"/>
+<label x="353.06" y="-248.92" size="1.778" layer="95" rot="R90"/>
 </segment>
 </net>
@@
 <label x="165.1" y="-147.32" size="1.778" layer="95"/>
 </segment>
-</net>
-<net name="VBAT" class="0">
-<segment>
-<pinref part="R22" gate="G$1" pin="2"/>
-<wire x1="287.02" y1="-30.48" x2="297.18" y2="-30.48" width="0.1524" layer="91"/>
-<label x="292.1" y="-30.48" size="1.778" layer="95"/>
-</segment>
-</net>
+<segment>
+<pinref part="STM32F1" gate="G$1" pin="PB0"/>
+<wire x1="368.3" y1="-330.2" x2="368.3" y2="-340.36" width="0.1524" layer="91"/>
+<label x="368.3" y="-340.36" size="1.778" layer="95" rot="R90"/>
+</segment>
+</net>

Commit message: Created PCB
Other:
- moved on the sheet: C10
Changed lines of the file:
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@@
 <layers>
 <layer number="1" name="Top" color="4" fill="1" visible="no" active="no"/>
+<layer number="2" name="Route2" color="1" fill="3" visible="no" active="no"/>
+<layer number="3" name="Route3" color="4" fill="3" visible="no" active="no"/>
+<layer number="4" name="Route4" color="1" fill="4" visible="no" active="no"/>
+<layer number="5" name="Route5" color="4" fill="4" visible="no" active="no"/>
+<layer number="6" name="Route6" color="1" fill="8" visible="no" active="no"/>
+<layer number="7" name="Route7" color="4" fill="8" visible="no" active="no"/>
+<layer number="8" name="Route8" color="1" fill="2" visible="no" active="no"/>
+<layer number="9" name="Route9" color="4" fill="2" visible="no" active="no"/>
+<layer number="10" name="Route10" color="1" fill="7" visible="no" active="no"/>
+<layer number="11" name="Route11" color="4" fill="7" visible="no" active="no"/>
+<layer number="12" name="Route12" color="1" fill="5" visible="no" active="no"/>
+<layer number="13" name="Route13" color="4" fill="5" visible="no" active="no"/>
+<layer number="14" name="Route14" color="1" fill="6" visible="no" active="no"/>
+<layer number="15" name="Route15" color="4" fill="6" visible="no" active="no"/>
 <layer number="16" name="Bottom" color="1" fill="1" visible="no" active="no"/>
 <layer number="17" name="Pads" color="2" fill="1" visible="no" active="no"/>
@@
 <part name="GND30" library="SUPPLY" deviceset="GND" device=""/>
 <part name="VBAT4" library="SUPPLY" deviceset="VBAT" device=""/>
+<part name="+3V8" library="SUPPLY" deviceset="+3V3" device=""/>
+<part name="+3V9" library="SUPPLY" deviceset="+3V3" device=""/>
+<part name="+3V11" library="SUPPLY" deviceset="+3V3" device=""/>
+<part name="P+4" library="SUPPLY" deviceset="+5V" device=""/>
+<part name="+3V12" library="SUPPLY" deviceset="+3V3" device=""/>
+<part name="+3V10" library="SUPPLY" deviceset="+3V3" device=""/>
 </parts>
 <sheets>
@@
 <attribute name="VALUE" x="283.464" y="-299.339" size="1.778" layer="96"/>
 </instance>
-<instance part="C10" gate="G$1" x="292.1" y="-309.88" smashed="yes">
-<attribute name="NAME" x="293.624" y="-306.959" size="1.778" layer="95"/>
-<attribute name="VALUE" x="293.624" y="-312.039" size="1.778" layer="96"/>
+<instance part="C10" gate="G$1" x="292.1" y="-312.42" smashed="yes">
+<attribute name="NAME" x="293.624" y="-309.499" size="1.778" layer="95"/>
+<attribute name="VALUE" x="293.624" y="-314.579" size="1.778" layer="96"/>
 </instance>
 <instance part="C11" gate="G$1" x="309.88" y="-259.08" smashed="yes">
@@
 <instance part="VBAT4" gate="G$1" x="299.72" y="-30.48" smashed="yes" rot="R270">
 <attribute name="VALUE" x="297.18" y="-27.94" size="1.778" layer="96"/>
+</instance>
+<instance part="+3V8" gate="G$1" x="309.88" y="-243.84" smashed="yes">
+<attribute name="VALUE" x="307.34" y="-248.92" size="1.778" layer="96" rot="R90"/>
+</instance>
+<instance part="+3V9" gate="G$1" x="426.72" y="-266.7" smashed="yes">
+<attribute name="VALUE" x="424.18" y="-271.78" size="1.778" layer="96" rot="R90"/>
+</instance>
+<instance part="+3V11" gate="G$1" x="347.98" y="-337.82" smashed="yes">
+<attribute name="VALUE" x="345.44" y="-342.9" size="1.778" layer="96" rot="R90"/>
+</instance>
+<instance part="P+4" gate="1" x="220.98" y="-22.86" smashed="yes" rot="R270">
+<attribute name="VALUE" x="215.9" y="-20.32" size="1.778" layer="96"/>
+</instance>
+<instance part="+3V12" gate="G$1" x="393.7" y="-332.74" smashed="yes">
+<attribute name="VALUE" x="391.16" y="-337.82" size="1.778" layer="96" rot="R90"/>
+</instance>
+<instance part="+3V10" gate="G$1" x="292.1" y="-299.72" smashed="yes">
+<attribute name="VALUE" x="289.56" y="-304.8" size="1.778" layer="96" rot="R90"/>
 </instance>
 </instances>
@@
 <pinref part="GND7" gate="1" pin="GND"/>
 <pinref part="C10" gate="G$1" pin="2"/>
-<wire x1="292.1" y1="-314.96" x2="292.1" y2="-312.42" width="0.1524" layer="91"/>
 </segment>
 <segment>
@@
 <wire x1="200.66" y1="-33.02" x2="210.82" y2="-33.02" width="0.1524" layer="91"/>
 <junction x="210.82" y="-33.02"/>
+<pinref part="P+4" gate="1" pin="+5V"/>
+<wire x1="210.82" y1="-22.86" x2="218.44" y2="-22.86" width="0.1524" layer="91"/>
 <junction x="210.82" y="-22.86"/>
-<wire x1="210.82" y1="-22.86" x2="218.44" y2="-22.86" width="0.1524" layer="91"/>
-<label x="215.9" y="-22.86" size="1.778" layer="95"/>
 </segment>
 <segment>
@@
 <pinref part="C11" gate="G$1" pin="1"/>
 <wire x1="309.88" y1="-248.92" x2="309.88" y2="-254" width="0.1524" layer="91"/>
-<label x="309.88" y="-243.84" size="1.778" layer="95" rot="R90"/>
-<wire x1="309.88" y1="-248.92" x2="309.88" y2="-243.84" width="0.1524" layer="91"/>
+<pinref part="+3V8" gate="G$1" pin="+3V3"/>
+<wire x1="309.88" y1="-248.92" x2="309.88" y2="-246.38" width="0.1524" layer="91"/>
 <junction x="309.88" y="-248.92"/>
-</segment>
-<segment>
-<pinref part="C10" gate="G$1" pin="1"/>
-<wire x1="292.1" y1="-304.8" x2="292.1" y2="-294.64" width="0.1524" layer="91"/>
-<pinref part="STM32F1" gate="G$1" pin="VDDA"/>
-<wire x1="327.66" y1="-304.8" x2="292.1" y2="-304.8" width="0.1524" layer="91"/>
-<junction x="292.1" y="-304.8"/>
-<label x="292.1" y="-299.72" size="1.778" layer="95" rot="R90"/>
-</segment>
-<segment>
-<pinref part="C5" gate="G$1" pin="1"/>
-<wire x1="347.98" y1="-342.9" x2="347.98" y2="-337.82" width="0.1524" layer="91"/>
-<label x="347.98" y="-342.9" size="1.778" layer="95" rot="R90"/>
-<pinref part="STM32F1" gate="G$1" pin="VDD_0"/>
-<wire x1="350.52" y1="-330.2" x2="350.52" y2="-342.9" width="0.1524" layer="91"/>
-<wire x1="350.52" y1="-342.9" x2="347.98" y2="-342.9" width="0.1524" layer="91"/>
-<junction x="347.98" y="-342.9"/>
-</segment>
-<segment>
-<pinref part="C7" gate="G$1" pin="1"/>
-<wire x1="393.7" y1="-340.36" x2="383.54" y2="-340.36" width="0.1524" layer="91"/>
-<pinref part="STM32F1" gate="G$1" pin="VDD_1"/>
-<wire x1="383.54" y1="-340.36" x2="383.54" y2="-330.2" width="0.1524" layer="91"/>
-<wire x1="393.7" y1="-340.36" x2="393.7" y2="-332.74" width="0.1524" layer="91"/>
-<junction x="393.7" y="-340.36"/>
-<label x="393.7" y="-337.82" size="1.778" layer="95" rot="R90"/>
 </segment>
 <segment>
@@
 <pinref part="C8" gate="G$1" pin="1"/>
 <wire x1="401.32" y1="-274.32" x2="426.72" y2="-274.32" width="0.1524" layer="91"/>
-<wire x1="426.72" y1="-274.32" x2="426.72" y2="-266.7" width="0.1524" layer="91"/>
+<pinref part="+3V9" gate="G$1" pin="+3V3"/>
+<wire x1="426.72" y1="-274.32" x2="426.72" y2="-269.24" width="0.1524" layer="91"/>
 <junction x="426.72" y="-274.32"/>
-<label x="426.72" y="-271.78" size="1.778" layer="95" rot="R90"/>
 </segment>
 <segment>
@@
 <wire x1="220.98" y1="-307.34" x2="220.98" y2="-320.04" width="0.1524" layer="91"/>
 </segment>
-</net>
+<segment>
+<pinref part="STM32F1" gate="G$1" pin="VDD_0"/>
+<wire x1="350.52" y1="-330.2" x2="350.52" y2="-340.36" width="0.1524" layer="91"/>
+<wire x1="350.52" y1="-340.36" x2="347.98" y2="-340.36" width="0.1524" layer="91"/>
+<pinref part="C5" gate="G$1" pin="1"/>
+<wire x1="347.98" y1="-340.36" x2="347.98" y2="-342.9" width="0.1524" layer="91"/>
+<pinref part="+3V11" gate="G$1" pin="+3V3"/>
+<junction x="347.98" y="-340.36"/>
+</segment>
+<segment>
+<pinref part="STM32F1" gate="G$1" pin="VDD_1"/>
+<wire x1="383.54" y1="-330.2" x2="383.54" y2="-337.82" width="0.1524" layer="91"/>
+<wire x1="383.54" y1="-337.82" x2="393.7" y2="-337.82" width="0.1524" layer="91"/>
+<pinref part="C7" gate="G$1" pin="1"/>
+<wire x1="393.7" y1="-337.82" x2="393.7" y2="-340.36" width="0.1524" layer="91"/>
+<pinref part="+3V12" gate="G$1" pin="+3V3"/>
+<wire x1="393.7" y1="-337.82" x2="393.7" y2="-335.28" width="0.1524" layer="91"/>
+<junction x="393.7" y="-337.82"/>
+</segment>
+<segment>
+<pinref part="C10" gate="G$1" pin="1"/>
+<pinref part="+3V10" gate="G$1" pin="+3V3"/>
+<wire x1="292.1" y1="-302.26" x2="292.1" y2="-304.8" width="0.1524" layer="91"/>
+<pinref part="STM32F1" gate="G$1" pin="VDDA"/>
+<wire x1="292.1" y1="-304.8" x2="292.1" y2="-307.34" width="0.1524" layer="91"/>
+<wire x1="327.66" y1="-304.8" x2="292.1" y2="-304.8" width="0.1524" layer="91"/>
+<junction x="292.1" y="-304.8"/>
+</segment>
+</net>

Commit message: handroute
Connections:
- removed net N$14: R5.1, R6.1, R7.1, R8.1
- net GND: now also R5.1, R6.1, R7.1, R8.1
Changed lines of the file:
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@@
 <part name="+3V12" library="SUPPLY" deviceset="+3V3" device=""/>
 <part name="+3V10" library="SUPPLY" deviceset="+3V3" device=""/>
+<part name="GND31" library="SUPPLY" deviceset="GND" device=""/>
 </parts>
 <sheets>
@@
 <instance part="+3V10" gate="G$1" x="292.1" y="-299.72" smashed="yes">
 <attribute name="VALUE" x="289.56" y="-304.8" size="1.778" layer="96" rot="R90"/>
+</instance>
+<instance part="GND31" gate="1" x="48.26" y="-76.2" smashed="yes">
+<attribute name="VALUE" x="46.99" y="-76.2" size="1.778" layer="96" rot="R90"/>
 </instance>
 </instances>
@@
 <wire x1="248.92" y1="-30.48" x2="259.08" y2="-30.48" width="0.1524" layer="91"/>
 </segment>
+<segment>
+<pinref part="GND31" gate="1" pin="GND"/>
+<wire x1="48.26" y1="-67.31" x2="48.26" y2="-73.66" width="0.1524" layer="91"/>
+<pinref part="R5" gate="G$1" pin="1"/>
+<wire x1="25.4" y1="-59.69" x2="25.4" y2="-67.31" width="0.1524" layer="91"/>
+<wire x1="25.4" y1="-67.31" x2="48.26" y2="-67.31" width="0.1524" layer="91"/>
+<pinref part="R6" gate="G$1" pin="1"/>
+<wire x1="48.26" y1="-67.31" x2="48.26" y2="-66.04" width="0.1524" layer="91"/>
+<wire x1="48.26" y1="-66.04" x2="48.26" y2="-59.69" width="0.1524" layer="91"/>
+<wire x1="48.26" y1="-67.31" x2="67.31" y2="-67.31" width="0.1524" layer="91"/>
+<junction x="48.26" y="-67.31"/>
+<pinref part="R7" gate="G$1" pin="1"/>
+<wire x1="67.31" y1="-67.31" x2="67.31" y2="-58.42" width="0.1524" layer="91"/>
+<wire x1="67.31" y1="-67.31" x2="86.36" y2="-67.31" width="0.1524" layer="91"/>
+<junction x="67.31" y="-67.31"/>
+<pinref part="R8" gate="G$1" pin="1"/>
+<wire x1="86.36" y1="-67.31" x2="86.36" y2="-58.42" width="0.1524" layer="91"/>
+</segment>
 </net>
 <net name="N$1" class="0">
@@
 </segment>
 </net>
-<net name="N$14" class="0">
-<segment>
-<pinref part="R5" gate="G$1" pin="1"/>
-<wire x1="25.4" y1="-59.69" x2="25.4" y2="-67.31" width="0.1524" layer="91"/>
-<wire x1="25.4" y1="-67.31" x2="48.26" y2="-67.31" width="0.1524" layer="91"/>
-<pinref part="R6" gate="G$1" pin="1"/>
-<wire x1="48.26" y1="-67.31" x2="48.26" y2="-59.69" width="0.1524" layer="91"/>
-<wire x1="48.26" y1="-67.31" x2="67.31" y2="-67.31" width="0.1524" layer="91"/>
-<junction x="48.26" y="-67.31"/>
-<pinref part="R7" gate="G$1" pin="1"/>
-<wire x1="67.31" y1="-67.31" x2="67.31" y2="-58.42" width="0.1524" layer="91"/>
-<wire x1="67.31" y1="-67.31" x2="86.36" y2="-67.31" width="0.1524" layer="91"/>
-<junction x="67.31" y="-67.31"/>
-<pinref part="R8" gate="G$1" pin="1"/>
-<wire x1="86.36" y1="-67.31" x2="86.36" y2="-58.42" width="0.1524" layer="91"/>
-</segment>
-</net>

Commit message: Fix errors
Connections:
- net +5V: no longer ZXMHC3_L.P1S/P2S, ZXMHC3_R.P1S/P2S
- net V+: now also ZXMHC3_L.P1S/P2S, ZXMHC3_R.P1S/P2S
Changed lines of the file:
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@@
 <part name="GND24" library="SUPPLY" deviceset="GND" device=""/>
 <part name="GND25" library="SUPPLY" deviceset="GND" device=""/>
-<part name="P+2" library="SUPPLY" deviceset="+5V" device=""/>
-<part name="P+3" library="SUPPLY" deviceset="+5V" device=""/>
 <part name="+3V4" library="SUPPLY" deviceset="+3V3" device=""/>
 <part name="+3V5" library="SUPPLY" deviceset="+3V3" device=""/>
@@
 <part name="+3V10" library="SUPPLY" deviceset="+3V3" device=""/>
 <part name="GND31" library="SUPPLY" deviceset="GND" device=""/>
+<part name="VBAT5" library="SUPPLY" deviceset="VBAT" device=""/>
+<part name="VBAT6" library="SUPPLY" deviceset="VBAT" device=""/>
 </parts>
 <sheets>
@@
 <attribute name="VALUE" x="219.71" y="-350.52" size="1.778" layer="96" rot="R90"/>
 </instance>
-<instance part="P+2" gate="1" x="187.96" y="-233.68" smashed="yes">
-<attribute name="VALUE" x="185.42" y="-238.76" size="1.778" layer="96" rot="R90"/>
-</instance>
-<instance part="P+3" gate="1" x="187.96" y="-299.72" smashed="yes">
-<attribute name="VALUE" x="185.42" y="-304.8" size="1.778" layer="96" rot="R90"/>
-</instance>
 <instance part="+3V4" gate="G$1" x="220.98" y="-233.68" smashed="yes">
 <attribute name="VALUE" x="218.44" y="-238.76" size="1.778" layer="96" rot="R90"/>
@@
 <instance part="GND31" gate="1" x="48.26" y="-76.2" smashed="yes">
 <attribute name="VALUE" x="46.99" y="-76.2" size="1.778" layer="96" rot="R90"/>
+</instance>
+<instance part="VBAT5" gate="G$1" x="187.96" y="-233.68" smashed="yes">
+<attribute name="VALUE" x="185.42" y="-236.22" size="1.778" layer="96" rot="R90"/>
+</instance>
+<instance part="VBAT6" gate="G$1" x="187.96" y="-299.72" smashed="yes">
+<attribute name="VALUE" x="185.42" y="-302.26" size="1.778" layer="96" rot="R90"/>
 </instance>
 </instances>
@@
 <junction x="363.22" y="-119.38"/>
 </segment>
-<segment>
-<pinref part="ZXMHC3_L" gate="G$1" pin="P1S/P2S"/>
-<wire x1="172.72" y1="-254" x2="187.96" y2="-254" width="0.1524" layer="91"/>
-<pinref part="P+2" gate="1" pin="+5V"/>
-<wire x1="187.96" y1="-236.22" x2="187.96" y2="-254" width="0.1524" layer="91"/>
-</segment>
-<segment>
-<pinref part="ZXMHC3_R" gate="G$1" pin="P1S/P2S"/>
-<wire x1="172.72" y1="-322.58" x2="187.96" y2="-322.58" width="0.1524" layer="91"/>
-<pinref part="P+3" gate="1" pin="+5V"/>
-<wire x1="187.96" y1="-322.58" x2="187.96" y2="-302.26" width="0.1524" layer="91"/>
-</segment>
 </net>
 <net name="V+" class="0">
@@
 <pinref part="VBAT4" gate="G$1" pin="V+"/>
 </segment>
-</net>
+<segment>
+<pinref part="ZXMHC3_L" gate="G$1" pin="P1S/P2S"/>
+<wire x1="172.72" y1="-254" x2="187.96" y2="-254" width="0.1524" layer="91"/>
+<wire x1="187.96" y1="-236.22" x2="187.96" y2="-254" width="0.1524" layer="91"/>
+<pinref part="VBAT5" gate="G$1" pin="V+"/>
+</segment>
+<segment>
+<pinref part="ZXMHC3_R" gate="G$1" pin="P1S/P2S"/>
+<wire x1="172.72" y1="-322.58" x2="187.96" y2="-322.58" width="0.1524" layer="91"/>
+<wire x1="187.96" y1="-322.58" x2="187.96" y2="-302.26" width="0.1524" layer="91"/>
+<pinref part="VBAT6" gate="G$1" pin="V+"/>
+</segment>
+</net>

Commit message: finished routing
Parts:
- C2: value 47 -> 47uF
Changed lines of the file:
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@@
 <part name="P+1" library="SUPPLY" deviceset="+5V" device=""/>
 <part name="C1" library="CAP_TANT_1210IN_3528MM" deviceset="CAP_TANT_1210IN_3528MM" device="" value="47uF"/>
-<part name="C2" library="CAP_TANT_1210IN_3528MM" deviceset="CAP_TANT_1210IN_3528MM" device="" value="47"/>
+<part name="C2" library="CAP_TANT_1210IN_3528MM" deviceset="CAP_TANT_1210IN_3528MM" device="" value="47uF"/>
 <part name="C3" library="CAP_CERAMIC_0805IN_2012MM" deviceset="CAP_CERAMIC_0805IN_2012MM" device="" value="10uF"/>
 <part name="C4" library="CAP_TANT_1210IN_3528MM" deviceset="CAP_TANT_1210IN_3528MM" device="" value="47uF"/>
